File: HDK/NVF2-SCS-Check-Indicate.kicad_pcb (KiCad board)
At the start: 2 copper layers, 80 x 50 mm, 39 parts, among them J101 Conn_01x02, J102 Conn_01x02, J103 Conn_01x02, J104 Conn_01x02, J105 SCS_IN, J106 Conn_01x02, Q101 2N7002, Q102 2N7002, Q103 2N7002, Q104 2N7002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

Commit message: rev1
Parts:
- C104, C105: footprint Capacitor_SMD:C_0603_1608Metric -> Capacitor_SMD:C_0805_2012Metric
- J101, J102, J103, J104, J106: footprint Connector_JST:JST_PH_S2B-PH-K_1x02_P2.00mm_Horizontal -> NVF-Kicad:PH_01x02H-H
- moved C104 0.23 mm to (125.3, 91.8)
- moved C105 0.23 mm to (127.6, 91.8)
Connections:
- SW102 pad 1: /~{SIG_TEST} -> Net-(R112-Pad2)
Routing:
- net /~{SIG_TEST}: track 101.5 -> 63.3 mm
- net Net-(R112-Pad2): track 2.83 -> 36.5 mm
- net GND: track 12.3 -> 10.00 mm, vias 25 -> 27
Other:
- board text added: "Scott CJX"

Commit message: updated
Parts:
- removed C102, C103, C110: 100n, Capacitor_SMD:C_0603_1608Metric
- removed C104: 2u2, Capacitor_SMD:C_0805_2012Metric
- removed R104, R105: 10k, Resistor_SMD:R_0603_1608Metric
- removed U102: MC14584B, Package_SO:SOIC-14_3.9x8.7mm_P1.27mm
- removed U103: MC14093B, Package_SO:SOIC-14_3.9x8.7mm_P1.27mm
- removed U104: MC14070B, Package_SO:SOIC-14_3.9x8.7mm_P1.27mm
- added C106: 2u2, Capacitor_SMD:C_0805_2012Metric, F.Cu at (128.6, 86.8)
- added C107: 2u2, Capacitor_SMD:C_0805_2012Metric, F.Cu at (128.6, 89.2)
- added D101: BAV70, Package_TO_SOT_SMD:SOT-23, F.Cu at (110.8, 89.9)
- added D102: LED, LED_SMD:LED_0603_1608Metric, F.Cu at (125.8, 80.2)
- added R113: 120, Resistor_SMD:R_1206_3216Metric, F.Cu at (156.8, 90.0)
- added R114: 10k, Resistor_SMD:R_0603_1608Metric, F.Cu at (145.3, 113.4)
- added R115: 1k, Resistor_SMD:R_0603_1608Metric, F.Cu at (146.9, 113.4)
- added RV101: 10K, NVF-Kicad:RV_Bourns_3362, F.Cu at (163.5, 84.0)
- added U105: AMS1117-5.0, Package_TO_SOT_SMD:SOT-223-3_TabPin2, F.Cu at (122.3, 89.2)
- C105: value 2u2 -> 100n; footprint Capacitor_SMD:C_0805_2012Metric -> Capacitor_SMD:C_0603_1608Metric
- R101, R102, R103: value 10k -> 14k
- R107, R108: value 120 -> 10k; footprint Resistor_SMD:R_1206_3216Metric -> Resistor_SMD:R_0603_1608Metric
- R109: value 120 -> 200; footprint Resistor_SMD:R_1206_3216Metric -> Resistor_SMD:R_0603_1608Metric
- R111: value 10k -> 120; footprint Resistor_SMD:R_0603_1608Metric -> Resistor_SMD:R_1206_3216Metric
- R112: value 1k -> 120; footprint Resistor_SMD:R_0603_1608Metric -> Resistor_SMD:R_1206_3216Metric
- SW101: value SW_Push_LED -> SW_Push; footprint NVF-Kicad:PH_01x04H-H -> NVF-Kicad:PushBtn_TS-1187A-B-A-B
- SW102: value SW_Push -> SW_Push_LED; footprint NVF-Kicad:PushBtn_TS-1187A-B-A-B -> NVF-Kicad:PH_01x04H-H
- U101: value AMS1117-5.0 -> ~; footprint Package_TO_SOT_SMD:SOT-223-3_TabPin2 -> Package_SO:SOIC-14_3.9x8.7mm_P1.27mm
- moved SW102 49.0 mm to (148.6, 118.2)
- moved SW101 41.9 mm to (140.0, 120.6), turned to -90 degrees
- moved G*** 41.4 mm to (129.8, 102.3), turned to 0 degrees
- moved Q105 38.4 mm to (149.6, 113.8), turned to -90 degrees
- moved R108 31.6 mm to (119.0, 107.4)
- moved C105 25.6 mm to (145.3, 110.3)
- moved R107 24.8 mm to (123.0, 107.4)
- moved R109 21.7 mm to (127.9, 80.3), turned to -90 degrees
- moved R112 21.5 mm to (149.6, 90.0), turned to 90 degrees
- moved R110 20.7 mm to (135.8, 90.0)
- moved U101 20.0 mm to (147.4, 101.2), turned to 0 degrees
- moved F101 16.9 mm to (118.0, 80.2), turned to 0 degrees
- moved R111 13.9 mm to (142.6, 90.0), turned to 90 degrees
- moved C101 9.66 mm to (150.2, 95.7)
- moved Q104 5.78 mm to (156.1, 85.6), turned to 90 degrees
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Connections:
- C105 pad 1: +5V -> /~{SIG_TEST}
- F101 pad 1: VCC -> Net-(D101-K)
- J105 pad 4: /SIG1_INV -> /SIG1
- J105 pad 6: /SIG2_INV -> /SIG2
- J105 pad 8: /SIG3_INV -> /SIG3
- J106 pad 2: /SIG_EZ1_IN -> /SIG4
- Q105 pad 1: /LED_TEST -> /~{SIG_TEST}
- R101 pad 1: +5V -> /SIG1_N
- R101 pad 2: /SIG1_N -> /SIG1
- R102 pad 1: +5V -> /SIG2_N
- R102 pad 2: /SIG2_N -> /SIG2
- R103 pad 1: +5V -> /SIG3_N
- R103 pad 2: /SIG3_N -> /SIG3
- R106 pad 1: /SIG1_INV -> /SIG3_N
- R107 pad 1: +12V -> /SIG2_N
- R107 pad 2: Net-(J101-Pin_1) -> GND
- R108 pad 1: +12V -> /SIG1_N
- R108 pad 2: Net-(J102-Pin_1) -> GND
- R109 pad 1: +12V -> GND
- R109 pad 2: Net-(J103-Pin_1) -> Net-(D102-K)
- R110 pad 1: +12V -> V_{LED}
- R110 pad 2: Net-(J104-Pin_1) -> Net-(J101-Pin_1)
- R111 pad 1: +5V -> V_{LED}
- R111 pad 2: /~{SIG_TEST} -> Net-(J102-Pin_1)
- R112 pad 1: /~{SIG_TEST} -> V_{LED}
- R112 pad 2: Net-(R112-Pad2) -> Net-(J103-Pin_1)
- SG101 pad L1: unconnected-(SG101C-V1-PadL1) -> VBUS
- SG101 pad R7: /SIG_EZ1_IN -> unconnected-(SG101C-PB12-PadR7)
- SG101 pad R8: unconnected-(SG101C-PB11-PadR8) -> /SIG4
- SW101 pad 1: Net-(R112-Pad2) -> /SIG_TEST
- SW102 pad 1: Net-(R112-Pad2) -> GND
- SW102 pad 2: GND -> /SIG_TEST
- U101 pad 1: GND -> /SIG1
- U101 pad 2: +5V -> /~{SIG_TEST}
- U101 pad 3: +12V -> /~{LED}1
Routing:
- net /LED_TEST: track 79.8 -> 0.00 mm
- net +12V: track 55.2 -> 104.6 mm, vias 5 -> 1
- net /SIG1_N: track 57.5 -> 9.75 mm, vias 1 -> 0
- net V_{LED}: track 0.00 -> 44.5 mm, vias 0 -> 4
- net /SIG3_N: track 46.0 -> 9.03 mm, vias 1 -> 0
- net Net-(R112-Pad2): track 36.5 -> 0.00 mm
- net /SIG2_N: track 44.3 -> 8.96 mm, vias 1 -> 0
- net /SIG3: track 15.4 -> 42.0 mm, vias 0 -> 2
- net /SIG1: track 18.2 -> 44.5 mm, vias 2 -> 0
- net /SIG3_INV: track 25.6 -> 0.00 mm, vias 2 -> 0
- net /SIG4: track 0.00 -> 23.8 mm, vias 0 -> 1
- net /SIG1_INV: track 23.1 -> 0.00 mm, vias 2 -> 0
- net /SIG_TEST: track 0.00 -> 20.8 mm
- net /SIG2: track 15.2 -> 35.1 mm, vias 2 -> 0
- net /SIG2_INV: track 17.7 -> 0.00 mm, vias 2 -> 0
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- removed copper zone on F.Cu, net +12V
- removed copper zone on F.Cu, net +5V
Other:
- board text added: "Indicators Rev 1"
- board text removed: "Multi SCS Detect Indicate"
- board text removed: "Rev1"
