File: HDK/NVF2-SCS-Check-Indicate.kicad_sch (KiCad schematic)
At the start: 41 parts, among them J101 Conn_01x02, J102 Conn_01x02, J103 Conn_01x02, J104 Conn_01x02, J105 SCS_IN, J106 Conn_01x02, Q101 2N7002, Q102 2N7002, Q103 2N7002, Q104 2N7002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

Commit message: rev1
Parts:
- C104: footprint Capacitor_SMD:C_0603_1608Metric -> Capacitor_SMD:C_0805_2012Metric; LCSC C1623 -> C377773
- C105: footprint Capacitor_SMD:C_0603_1608Metric -> Capacitor_SMD:C_0805_2012Metric; LCSC C14663 -> C377773
- C106, C107, C108: footprint Capacitor_THT:CP_Radial_D10.0mm_P5.00mm -> (none)
- J101, J102, J103, J104, J106: footprint Connector_JST:JST_PH_S2B-PH-K_1x02_P2.00mm_Horizontal -> NVF-Kicad:PH_01x02H-H
- SW101: footprint NVF-Kicad:PH_01x04H-H -> (none)
- SW102: LCSC (none) -> C318884
- U101: LCSC (none) -> C6187
- U102: Element14 (none) -> 9665102
Connections:
- net ~{SIG_TEST}: no longer SW102.1
- net at R112.2, SW101.1: now also SW102.1
Other:
- moved on the sheet: SW102

Commit message: updated
Parts:
- removed C101, C102, C103, C110: 100n, Capacitor_SMD:C_0603_1608Metric, symbol Device:C
- removed C104: 2u2, Capacitor_SMD:C_0805_2012Metric, symbol Device:C
- removed C108: 470u, symbol Device:C
- removed C109: 10u, symbol Device:C
- removed R111: 10k, Resistor_SMD:R_0603_1608Metric, symbol Device:R
- removed R112: 1k, Resistor_SMD:R_0603_1608Metric, symbol Device:R
- removed SW101: SW_Push_LED, symbol Switch:SW_Push_LED
- removed SW102: SW_Push, NVF-Kicad:PushBtn_TS-1187A-B-A-B, symbol Switch:SW_Push
- removed U101: AMS1117-5.0, Package_TO_SOT_SMD:SOT-223-3_TabPin2, symbol Regulator_Linear:AMS1117-5.0
- removed U102: MC14584B, Package_SO:SOIC-14_3.9x8.7mm_P1.27mm, symbol NVF-Kicad:HEX_NOT
- removed U103: MC14093B, Package_SO:SOIC-14_3.9x8.7mm_P1.27mm, symbol NVF-Kicad:QUAD_NAND
- removed U104: MC14070B, Package_SO:SOIC-14_3.9x8.7mm_P1.27mm, symbol NVF-Kicad:QUAD_XOR
- added C101: 100n, Capacitor_SMD:C_0603_1608Metric, symbol Device:C_Small
- added D101: BAV70, Package_TO_SOT_SMD:SOT-23, symbol Diode:BAV70
- added D102: LED, LED_SMD:LED_0603_1608Metric, symbol Device:LED
- added R104: 14k, Resistor_SMD:R_0603_1608Metric, symbol Device:R
- added R105, R114: 10k, Resistor_SMD:R_0603_1608Metric, symbol Device:R
- added R109: 200, Resistor_SMD:R_0603_1608Metric, symbol Device:R
- added R115: 1k, Resistor_SMD:R_0603_1608Metric, symbol Device:R
- added RV101: 10K, NVF-Kicad:RV_Bourns_3362, symbol Device:R_Potentiometer
- added SW101: SW_Push, NVF-Kicad:PushBtn_TS-1187A-B-A-B, symbol Switch:SW_Push
- added SW102: SW_Push_LED, NVF-Kicad:PH_01x04H-H, symbol Switch:SW_Push_LED
- added U101: ~, Package_SO:SOIC-14_3.9x8.7mm_P1.27mm, symbol NVF-Kicad:QUAD_XOR
- added U105: AMS1117-5.0, Package_TO_SOT_SMD:SOT-223-3_TabPin2, symbol Regulator_Linear:AMS1117-5.0
- C105: value 2u2 -> 100n; footprint Capacitor_SMD:C_0805_2012Metric -> Capacitor_SMD:C_0603_1608Metric; LCSC C377773 -> C14663
- C106, C107: value 470u -> 2u2; footprint (none) -> Capacitor_SMD:C_0805_2012Metric; LCSC (none) -> C377773; now fitted
- J105, SG101: LCSC (none) -> -
- R101, R102, R103: value 10k -> 14k
- R106: renamed from R104; LCSC (none) -> C25804
- R107: renamed from R105; LCSC (none) -> C25804
- R108: renamed from R106; LCSC (none) -> C25804
- R110: renamed from R107; LCSC (none) -> C17909
- R111: renamed from R108; LCSC (none) -> C17909
- R112: renamed from R109; LCSC (none) -> C17909
- R113: renamed from R110; LCSC (none) -> C17909
Connections:
- net LED_TEST is gone; now on net ~{SIG_TEST}: Q105.1 (G)
- net +12V: now also C106.1, D102.2 (A), RV101.1, SW102.4 (A), U105.3 (VI); no longer R110.1, R111.1, R112.1, R113.1
- net +5V: now also C107.1, C101.1, R114.1, U101.14 (VDD), U105.2 (VO); no longer C105.1, R101.1, R102.1, R103.1
- net GND: now also C101.2, R105.2, R109.1, RV101.3, SW101.2, SW102.1, U101.7 (VSS), U105.1 (GND)
- net LED_TEST-: now also SW102.3 (K)
- net SIG1: now also J105.4 (Pin_4), R101.2, U101.1 (IN_1A)
- net SIG1_N: now also R101.1, R108.1; no longer R101.2
- net SIG2: now also J105.6 (Pin_6), R102.2, U101.5 (IN_1B)
- net SIG2_N: now also R102.1, R107.1; no longer R102.2
- net SIG3: now also J105.8 (Pin_8), R103.2, U101.12 (IN_2C)
- net SIG3_N: now also R103.1, R106.1; no longer R103.2
- net VCC: now also D101.1 (A); no longer F101.1
- net ~{SIG_TEST}: now also C105.1, R114.2, R115.1, U101.10 (IN_1D), U101.11 (IN_1C), U101.2 (IN_2A), U101.6 (IN_2B)
- net VBUS: now reaches SG101.L1 (V1)
- net VBUS: now also D101.2 (A)
- net SIG4: now reaches SG101.R8 (PB11)
- net SIG4: now also J106.2 (Pin_2), R104.2, U101.8 (IN_2D)
- net at J102.1 (Pin_1), Q102.3 (D), R111.2: no longer C107.1
- net at J101.1 (Pin_1), Q101.3 (D), R110.2: no longer C106.1
- removed net SIG1_INV: J105.4 (Pin_4), R108.1
- net SIG1_OUT renamed ~{LED}1
- net ~{LED}1: now also U101.3 (OUTA)
- removed net SIG2_INV: J105.6 (Pin_6), R107.1
- net SIG2_OUT renamed ~{LED}2
- net ~{LED}2: now also U101.4 (OUTB)
- removed net SIG3_INV: J105.8 (Pin_8), R106.1
- net SIG3_OUT renamed ~{LED}3
- net ~{LED}3: now also U101.13 (OUTC)
- net SIG4_OUT renamed ~{LED}4
- net ~{LED}4: now also U101.9 (OUTD)
- net SIG_EZ1_IN: no longer names the net of SG101.R7 (PB12)
- net SIG_EZ1_IN: no longer J106.2 (Pin_2)
- new net: D101.3 (K), F101.1
- new net: D102.1 (K), R109.2
- new net SIG4_N: R104.1, R105.1
- new net SIG_TEST: R115.2, SW101.1, SW102.2
- new net V_{LED}: R110.1, R111.1, R112.1, RV101.2
- no-connect marks 18 -> 12
Other:
- note added: "Board Connections"
- note added: "Board Interconnect"
- note added: "SIG* Does NOT have Voltage Divider SIG*_N Has Voltage Divider"
- note added: "Signal Handling"
- note added: "Signal Logic"
- note added: "Test"
- note removed: "Non-SCS"
- note removed: "SIG_N: Normal Signal pulled-up by default. SIG_INV: Inverted Signal pulled-down by default."
- moved on the sheet: J101, J102, J103, J104, J105, J106, Q101, Q102, Q103, Q104, Q105, R106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
